Commit message: added mtc and updated tool link

File: rg2_description/urdf/rg2_gripper.urdf.xacro (robot description, xacro)
@@ -306,6 +306,6 @@
         </joint>
         <joint name="${prefix}-tool_joint" type="fixed">
-            <!--default toolframe - X+ left, Y+ up, Z+ front-->
-            <origin xyz="0.2 0 0" rpy="${pi/2} 0 ${pi/2}"/>
+            <!--default toolframe - X+ up, Y+ right, Z+ front-->
+            <origin xyz="0.2 0 0" rpy="${pi/2} ${pi/2} ${pi/2}"/>
             <parent link="${prefix}_hand_link"/>
             <child link="${prefix}_tool_link"/>

Commit message: adjusted the tool joint

File: rg2_description/urdf/rg2_gripper.urdf.xacro (robot description, xacro)
@@ -307,5 +307,5 @@
         <joint name="${prefix}-tool_joint" type="fixed">
             <!--default toolframe - X+ up, Y+ right, Z+ front-->
-            <origin xyz="0.2 0 0" rpy="${pi/2} ${pi/2} ${pi/2}"/>
+            <origin xyz="0.1 0 0" rpy="${pi/2} ${pi/2} ${pi/2}"/>
             <parent link="${prefix}_hand_link"/>
             <child link="${prefix}_tool_link"/>
